Commit message: fix: correct chassis mesh orientation, wheel positions and IR sensor placement in Rwiz

File: slodda_description/urdf/slodda_real.urdf.xacro (robot description, xacro)
@@ -1,28 +1,25 @@
 <?xml version="1.0"?>
 <robot xmlns:xacro="http://www.ros.org/wiki/xacro" name="slodda">
-  <!-- Properties -->
   <xacro:property name="chassis_length" value="0.250"/>
-  <xacro:property name="chassis_width" value="0.280"/>
+  <xacro:property name="chassis_width"  value="0.280"/>
   <xacro:property name="chassis_height" value="0.122"/>
-  <xacro:property name="chassis_mass" value="2.5"/>
-  <xacro:property name="wheel_radius" value="0.045"/>
-  <xacro:property name="wheel_width" value="0.04"/>
-  <xacro:property name="track_separation" value="0.280"/>
-  <xacro:property name="ir_sensor_range_min" value="0.04"/>
-  <xacro:property name="ir_sensor_range_max" value="0.30"/>
-  <!-- Materials -->
-  <material name="orange">
-    <color rgba="0.8 0.4 0.1 1.0"/>
-  </material>
-  <material name="blue">
-    <color rgba="0.2 0.4 0.8 1.0"/>
-  </material>
-  <material name="grey">
-    <color rgba="0.5 0.5 0.5 1.0"/>
-  </material>
-  <!-- Base link (chassis with mesh) -->
+  <xacro:property name="chassis_mass"   value="2.5"/>
+  <xacro:property name="wheel_radius"   value="0.045"/>
+  <xacro:property name="wheel_width"    value="0.035"/>
+  <xacro:property name="wheel_x_offset" value="0.090"/>
+  <xacro:property name="wheel_y_offset" value="0.123"/>
+  <material name="orange">   <color rgba="0.8 0.4 0.1 1.0"/> </material>
+  <material name="dark_grey"><color rgba="0.2 0.2 0.2 1.0"/> </material>
+  <material name="grey">     <color rgba="0.5 0.5 0.5 1.0"/> </material>
+  <link name="base_footprint"/>
+  <joint name="base_footprint_joint" type="fixed">
+    <parent link="base_footprint"/>
+    <child link="base_link"/>
+    <origin xyz="0 0 ${wheel_radius}" rpy="0 0 0"/>
+  </joint>
+  <!-- CHASSIS: enkel boks, ingen mesh -->
   <link name="base_link">
     <visual>
-      <origin xyz="0 0 0" rpy="0 0 0"/>
+      <origin xyz="0.1414 0.1000 0.0" rpy="${pi/2} 0 ${pi}"/>
       <geometry>
         <mesh filename="package://slodda_description/meshes/chassis.stl" scale="0.001 0.001 0.001"/>
@@ -31,12 +28,12 @@
     </visual>
     <collision>
-      <origin xyz="0 0 0.061" rpy="0 0 0"/>
+      <origin xyz="0.1414 0.1000 0.0" rpy="${pi/2} 0 ${pi}"/>
       <geometry>
-        <box size="${chassis_length} ${chassis_width} ${chassis_height}"/>
+        <mesh filename="package://slodda_description/meshes/chassis.stl" scale="0.001 0.001 0.001"/>
       </geometry>
     </collision>
     <inertial>
       <mass value="${chassis_mass}"/>
-      <origin xyz="0 0 0.061" rpy="0 0 0"/>
+      <origin xyz="0.1414 0.1000 0.0" rpy="${pi/2} 0 ${pi}"/>
       <inertia ixx="0.052" ixy="0.0" ixz="0.0"
                iyy="0.046" iyz="0.0"
@@ -44,149 +41,75 @@
     </inertial>
   </link>
-  <!-- Left track (simplified as single cylinder) -->
-  <link name="left_track">
-    <visual>
-      <origin xyz="0 0 0" rpy="1.5708 0 0"/>
-      <geometry>
-        <cylinder radius="${wheel_radius}" length="${chassis_length}"/>
-      </geometry>
-      <material name="blue"/>
-    </visual>
-    <collision>
-      <origin xyz="0 0 0" rpy="1.5708 0 0"/>
-      <geometry>
-        <cylinder radius="${wheel_radius}" length="${chassis_length}"/>
-      </geometry>
-    </collision>
-    <inertial>
-      <mass value="0.5"/>
-      <origin xyz="0 0 0" rpy="1.5708 0 0"/>
-      <inertia ixx="0.002" ixy="0.0" ixz="0.0"
-               iyy="0.002" iyz="0.0"
-               izz="0.001"/>
-    </inertial>
-  </link>
-  <joint name="left_track_joint" type="continuous">
-    <parent link="base_link"/>
-    <child link="left_track"/>
-    <origin xyz="0 ${track_separation/2} ${wheel_radius}" rpy="0 0 0"/>
-    <axis xyz="0 1 0"/>
-  </joint>
-  <!-- Right track (simplified as single cylinder) -->
-  <link name="right_track">
-    <visual>
-      <origin xyz="0 0 0" rpy="1.5708 0 0"/>
-      <geometry>
-        <cylinder radius="${wheel_radius}" length="${chassis_length}"/>
-      </geometry>
-      <material name="blue"/>
-    </visual>
-    <collision>
-      <origin xyz="0 0 0" rpy="1.5708 0 0"/>
-      <geometry>
-        <cylinder radius="${wheel_radius}" length="${chassis_length}"/>
-      </geometry>
-    </collision>
-    <inertial>
-      <mass value="0.5"/>
-      <origin xyz="0 0 0" rpy="1.5708 0 0"/>
-      <inertia ixx="0.002" ixy="0.0" ixz="0.0"
-               iyy="0.002" iyz="0.0"
-               izz="0.001"/>
-    </inertial>
-  </link>
-  <joint name="right_track_joint" type="continuous">
-    <parent link="base_link"/>
-    <child link="right_track"/>
-    <origin xyz="0 ${-track_separation/2} ${wheel_radius}" rpy="0 0 0"/>
-    <axis xyz="0 1 0"/>
-  </joint>
-  <!-- IR Sensor - Front Left -->
-  <link name="ir_front_left">
-    <visual>
-      <geometry>
-        <box size="0.02 0.01 0.01"/>
-      </geometry>
-      <material name="grey"/>
-    </visual>
-    <collision>
-      <geometry>
-        <box size="0.02 0.01 0.01"/>
-      </geometry>
-    </collision>
-    <inertial>
-      <mass value="0.01"/>
-      <inertia ixx="0.00001" ixy="0.0" ixz="0.0"
-               iyy="0.00001" iyz="0.0"
-               izz="0.00001"/>
-    </inertial>
-  </link>
-  <joint name="ir_front_left_joint" type="fixed">
-    <parent link="base_link"/>
-    <child link="ir_front_left"/>
-    <origin xyz="0.125 0.08 0.08" rpy="0 0 0.3"/>
-  </joint>
-  <!-- IR Sensor - Front Center -->
-  <link name="ir_front_center">
-    <visual>
-      <geometry>
-        <box size="0.02 0.01 0.01"/>
-      </geometry>
-      <material name="grey"/>
-    </visual>
-    <collision>
-      <geometry>
-        <box size="0.02 0.01 0.01"/>
-      </geometry>
-    </collision>
-    <inertial>
-      <mass value="0.01"/>
-      <inertia ixx="0.00001" ixy="0.0" ixz="0.0"
-               iyy="0.00001" iyz="0.0"
-               izz="0.00001"/>
-    </inertial>
-  </link>
-  <joint name="ir_front_center_joint" type="fixed">
-    <parent link="base_link"/>
-    <child link="ir_front_center"/>
-    <origin xyz="0.125 0 0.08" rpy="0 0 0"/>
-  </joint>
-  <!-- IR Sensor - Front Right -->
-  <link name="ir_front_right">
-    <visual>
-      <geometry>
-        <box size="0.02 0.01 0.01"/>
-      </geometry>
-      <material name="grey"/>
-    </visual>
-    <collision>
-      <geometry>
-        <box size="0.02 0.01 0.01"/>
-      </geometry>
-    </collision>
-    <inertial>
-      <mass value="0.01"/>
-      <inertia ixx="0.00001" ixy="0.0" ixz="0.0"
-               iyy="0.00001" iyz="0.0"
-               izz="0.00001"/>
-    </inertial>
-  </link>
-  <joint name="ir_front_right_joint" type="fixed">
-    <parent link="base_link"/>
-    <child link="ir_front_right"/>
-    <origin xyz="0.125 -0.08 0.08" rpy="0 0 -0.3"/>
-  </joint>
-  <!-- Gazebo Plugins -->
-  <!-- Differential Drive Plugin with DFRobot motor specs -->
+  <xacro:macro name="wheel" params="name x y">
+    <link name="${name}">
+      <visual>
+        <origin xyz="0 0 0" rpy="${pi/2} 0 0"/>
+        <geometry>
+          <cylinder radius="${wheel_radius}" length="${wheel_width}"/>
+        </geometry>
+        <material name="dark_grey"/>
+      </visual>
+      <collision>
+        <origin xyz="0 0 0" rpy="${pi/2} 0 0"/>
+        <geometry>
+          <cylinder radius="${wheel_radius}" length="${wheel_width}"/>
+        </geometry>
+      </collision>
+      <inertial>
+        <mass value="0.15"/>
+        <origin xyz="0 0 0"/>
+        <inertia ixx="0.0001" ixy="0.0" ixz="0.0"
+                 iyy="0.0001" iyz="0.0"
+                 izz="0.0002"/>
+      </inertial>
+    </link>
+    <joint name="${name}_joint" type="continuous">
+      <parent link="base_link"/>
+      <child link="${name}"/>
+      <origin xyz="${x} ${y} 0" rpy="0 0 0"/>
+      <axis xyz="0 1 0"/>
+    </joint>
+  </xacro:macro>
+  <xacro:wheel name="left_front_wheel"  x=" ${wheel_x_offset}" y=" ${wheel_y_offset}"/>
+  <xacro:wheel name="left_rear_wheel"   x="-${wheel_x_offset}" y=" ${wheel_y_offset}"/>
+  <xacro:wheel name="right_front_wheel" x=" ${wheel_x_offset}" y="-${wheel_y_offset}"/>
+  <xacro:wheel name="right_rear_wheel"  x="-${wheel_x_offset}" y="-${wheel_y_offset}"/>
+  <xacro:macro name="ir_sensor" params="name x y yaw">
+    <link name="${name}">
+      <visual>
+        <geometry><box size="0.02 0.01 0.01"/></geometry>
+        <material name="grey"/>
+      </visual>
+      <collision>
+        <geometry><box size="0.02 0.01 0.01"/></geometry>
+      </collision>
+      <inertial>
+        <mass value="0.01"/>
+        <origin xyz="0 0 0"/>
+        <inertia ixx="0.00001" ixy="0.0" ixz="0.0"
+                 iyy="0.00001" iyz="0.0"
+                 izz="0.00001"/>
+      </inertial>
+    </link>
+    <joint name="${name}_joint" type="fixed">
+      <parent link="base_link"/>
+      <child link="${name}"/>
+      <origin xyz="${x} ${y} 0.04" rpy="0 0 ${yaw}"/>
+    </joint>
+  </xacro:macro>
+  <xacro:ir_sensor name="ir_front_left"   x="-0.135" y=" 0.07" yaw=" 0.3"/>
+  <xacro:ir_sensor name="ir_front_center" x="-0.135" y=" 0.00" yaw=" 0.0"/>
+  <xacro:ir_sensor name="ir_front_right"  x="-0.135" y="-0.07" yaw="-0.3"/>
   <gazebo>
-    <plugin filename="gz-sim-diff-drive-system" name="gz::sim::systems::DiffDrive">
-      <left_joint>left_track_joint</left_joint>
-      <right_joint>right_track_joint</right_joint>
-      <wheel_separation>${track_separation}</wheel_separation>
+    <plugin filename="gz-sim-diff-drive-system"
+            name="gz::sim::systems::DiffDrive">
+      <left_joint>left_rear_wheel_joint</left_joint>
+      <right_joint>right_rear_wheel_joint</right_joint>
+      <wheel_separation>${wheel_y_offset * 2}</wheel_separation>
       <wheel_radius>${wheel_radius}</wheel_radius>
+      <max_linear_velocity>0.5</max_linear_velocity>
+      <max_angular_velocity>1.0</max_angular_velocity>
       <max_linear_acceleration>1.0</max_linear_acceleration>
       <max_angular_acceleration>2.0</max_angular_acceleration>
-      <max_linear_velocity>0.5</max_linear_velocity>
-      <max_angular_velocity>1.0</max_angular_velocity>
       <odom_publish_frequency>50</odom_publish_frequency>
       <topic>cmd_vel</topic>
@@ -196,90 +119,14 @@
     </plugin>
   </gazebo>
-  <!-- IR Sensor Plugins (Sharp GP2Y0A41SK0F - 4-30cm range) -->
-  <gazebo reference="ir_front_left">
-    <sensor name="ir_front_left_sensor" type="gpu_lidar">
-      <update_rate>10</update_rate>
-      <lidar>
-        <scan>
-          <horizontal>
-            <samples>5</samples>
-            <resolution>1</resolution>
-            <min_angle>-0.1</min_angle>
-            <max_angle>0.1</max_angle>
-          </horizontal>
-        </scan>
-        <range>
-          <min>${ir_sensor_range_min}</min>
-          <max>${ir_sensor_range_max}</max>
-          <resolution>0.01</resolution>
-        </range>
-      </lidar>
-      <always_on>1</always_on>
-      <visualize>true</visualize>
-      <topic>ir_front_left</topic>
-    </sensor>
-  </gazebo>
-  <gazebo reference="ir_front_center">
-    <sensor name="ir_front_center_sensor" type="gpu_lidar">
-      <update_rate>10</update_rate>
-      <lidar>
-        <scan>
-          <horizontal>
-            <samples>5</samples>
-            <resolution>1</resolution>
-            <min_angle>-0.1</min_angle>
-            <max_angle>0.1</max_angle>
-          </horizontal>
-        </scan>
-        <range>
-          <min>${ir_sensor_range_min}</min>
-          <max>${ir_sensor_range_max}</max>
-          <resolution>0.01</resolution>
-        </range>
-      </lidar>
-      <always_on>1</always_on>
-      <visualize>true</visualize>
-      <topic>ir_front_center</topic>
-    </sensor>
-  </gazebo>
-  <gazebo reference="ir_front_right">
-    <sensor name="ir_front_right_sensor" type="gpu_lidar">
-      <update_rate>10</update_rate>
-      <lidar>
-        <scan>
-          <horizontal>
-            <samples>5</samples>
-            <resolution>1</resolution>
-            <min_angle>-0.1</min_angle>
-            <max_angle>0.1</max_angle>
-          </horizontal>
-        </scan>
-        <range>
-          <min>${ir_sensor_range_min}</min>
-          <max>${ir_sensor_range_max}</max>
-          <resolution>0.01</resolution>
-        </range>
-      </lidar>
-      <always_on>1</always_on>
-      <visualize>true</visualize>
-      <topic>ir_front_right</topic>
-    </sensor>
-  </gazebo>
-  <!-- Track friction -->
-  <gazebo reference="left_track">
-    <mu1>1.0</mu1>
-    <mu2>1.0</mu2>
-    <kp>1000000.0</kp>
-    <kd>100.0</kd>
-    <minDepth>0.001</minDepth>
-    <maxVel>1.0</maxVel>
-  </gazebo>
-  <gazebo reference="right_track">
-    <mu1>1.0</mu1>
-    <mu2>1.0</mu2>
-    <kp>1000000.0</kp>
-    <kd>100.0</kd>
-    <minDepth>0.001</minDepth>
-    <maxVel>1.0</maxVel>
-  </gazebo>
+  <xacro:macro name="wheel_gazebo" params="name">
+    <gazebo reference="${name}">
+      <mu1>1.5</mu1><mu2>1.5</mu2>
+      <kp>1000000.0</kp><kd>100.0</kd>
+      <minDepth>0.001</minDepth><maxVel>1.0</maxVel>
+    </gazebo>
+  </xacro:macro>
+  <xacro:wheel_gazebo name="left_front_wheel"/>
+  <xacro:wheel_gazebo name="left_rear_wheel"/>
+  <xacro:wheel_gazebo name="right_front_wheel"/>
+  <xacro:wheel_gazebo name="right_rear_wheel"/>
 </robot>

Commit message: feat: working simulation with skid-steer, arena and sensor plugins attempt

File: slodda_description/urdf/slodda_real.urdf.xacro (robot description, xacro)
@@ -28,15 +28,15 @@
     </visual>
     <collision>
-      <origin xyz="0.1414 0.1000 0.0" rpy="${pi/2} 0 ${pi}"/>
+      <origin xyz="0 0 0.061" rpy="0 0 0"/>
       <geometry>
-        <mesh filename="package://slodda_description/meshes/chassis.stl" scale="0.001 0.001 0.001"/>
+        <box size="${chassis_length} ${chassis_width} ${chassis_height}"/>
       </geometry>
     </collision>
     <inertial>
       <mass value="${chassis_mass}"/>
-      <origin xyz="0.1414 0.1000 0.0" rpy="${pi/2} 0 ${pi}"/>
-      <inertia ixx="0.052" ixy="0.0" ixz="0.0"
-               iyy="0.046" iyz="0.0"
-               izz="0.078"/>
+      <origin xyz="0 0 0.061" rpy="0 0 0"/>
+      <inertia ixx="0.0197" ixy="0.0" ixz="0.0"
+               iyy="0.0164" iyz="0.0"
+               izz="0.0309"/>
     </inertial>
   </link>
@@ -68,5 +68,5 @@
       <child link="${name}"/>
       <origin xyz="${x} ${y} 0" rpy="0 0 0"/>
-      <axis xyz="0 1 0"/>
+      <axis xyz="0 -1 0"/>
     </joint>
   </xacro:macro>
@@ -97,4 +97,7 @@
       <origin xyz="${x} ${y} 0.04" rpy="0 0 ${yaw}"/>
     </joint>
+    <gazebo reference="${name}_joint">
+      <preserveFixedJoint>true</preserveFixedJoint>
+    </gazebo>
   </xacro:macro>
   <xacro:ir_sensor name="ir_front_left"   x="-0.135" y=" 0.07" yaw=" 0.3"/>
@@ -104,5 +107,7 @@
     <plugin filename="gz-sim-diff-drive-system"
             name="gz::sim::systems::DiffDrive">
+      <left_joint>left_front_wheel_joint</left_joint>
       <left_joint>left_rear_wheel_joint</left_joint>
+      <right_joint>right_front_wheel_joint</right_joint>
       <right_joint>right_rear_wheel_joint</right_joint>
       <wheel_separation>${wheel_y_offset * 2}</wheel_separation>
@@ -130,3 +135,32 @@
   <xacro:wheel_gazebo name="right_front_wheel"/>
   <xacro:wheel_gazebo name="right_rear_wheel"/>
+  <!-- IR Sensor Plugins -->
+  <xacro:macro name="ir_gazebo" params="name topic">
+    <gazebo reference="${name}">
+      <sensor name="${name}_sensor" type="gpu_lidar">
+        <update_rate>10</update_rate>
+        <lidar>
+          <scan>
+            <horizontal>
+              <samples>5</samples>
+              <resolution>1</resolution>
+              <min_angle>-0.1</min_angle>
+              <max_angle>0.1</max_angle>
+            </horizontal>
+          </scan>
+          <range>
+            <min>0.04</min>
+            <max>0.30</max>
+            <resolution>0.01</resolution>
+          </range>
+        </lidar>
+        <always_on>1</always_on>
+        <visualize>true</visualize>
+        <topic>${topic}</topic>
+      </sensor>
+    </gazebo>
+  </xacro:macro>
+  <xacro:ir_gazebo name="ir_front_left"   topic="ir_front_left"/>
+  <xacro:ir_gazebo name="ir_front_center" topic="ir_front_center"/>
+  <xacro:ir_gazebo name="ir_front_right"  topic="ir_front_right"/>
 </robot>

Commit message: fix: working IR sensors and obstacle avoidance
- Switch to gpu_lidar sensor type (lidar not supported in Harmonic)
- Use ogre2 server + ogre GUI render engines (fixes Intel GPU issues)
- Remove preserveFixedJoint from IR sensor links (caused sensors to
  stay at world origin instead of following robot)
- Add obstacle_avoider node with reactive state machine
- IR sensors now correctly read inf (free) and ~0.13m (near wall)

File: slodda_description/urdf/slodda_real.urdf.xacro (robot description, xacro)
@@ -18,5 +18,4 @@
     <origin xyz="0 0 ${wheel_radius}" rpy="0 0 0"/>
   </joint>
-  <!-- CHASSIS: enkel boks, ingen mesh -->
   <link name="base_link">
     <visual>
@@ -75,4 +74,5 @@
   <xacro:wheel name="right_front_wheel" x=" ${wheel_x_offset}" y="-${wheel_y_offset}"/>
   <xacro:wheel name="right_rear_wheel"  x="-${wheel_x_offset}" y="-${wheel_y_offset}"/>
+  <!-- IR sensor lenker - ingen preserveFixedJoint, slik at de lumpes inn i base_link -->
   <xacro:macro name="ir_sensor" params="name x y yaw">
     <link name="${name}">
@@ -81,13 +81,10 @@
         <material name="grey"/>
       </visual>
-      <collision>
-        <geometry><box size="0.02 0.01 0.01"/></geometry>
-      </collision>
       <inertial>
-        <mass value="0.01"/>
+        <mass value="0.001"/>
         <origin xyz="0 0 0"/>
-        <inertia ixx="0.00001" ixy="0.0" ixz="0.0"
-                 iyy="0.00001" iyz="0.0"
-                 izz="0.00001"/>
+        <inertia ixx="0.000001" ixy="0.0" ixz="0.0"
+                 iyy="0.000001" iyz="0.0"
+                 izz="0.000001"/>
       </inertial>
     </link>
@@ -95,13 +92,39 @@
       <parent link="base_link"/>
       <child link="${name}"/>
-      <origin xyz="${x} ${y} 0.04" rpy="0 0 ${yaw}"/>
+      <origin xyz="${x} ${y} 0.13" rpy="0 0 ${yaw}"/>
     </joint>
-    <gazebo reference="${name}_joint">
-      <preserveFixedJoint>true</preserveFixedJoint>
-    </gazebo>
   </xacro:macro>
   <xacro:ir_sensor name="ir_front_left"   x="-0.135" y=" 0.07" yaw="${pi - 0.3}"/>
   <xacro:ir_sensor name="ir_front_center" x="-0.135" y=" 0.00" yaw="${pi}"/>
   <xacro:ir_sensor name="ir_front_right"  x="-0.135" y="-0.07" yaw="${pi + 0.3}"/>
+  <!-- IR sensor plugins -->
+  <xacro:macro name="ir_gazebo" params="name topic">
+    <gazebo reference="${name}">
+      <sensor name="${name}_sensor" type="gpu_lidar">
+        <update_rate>10</update_rate>
+        <lidar>
+          <scan>
+            <horizontal>
+              <samples>5</samples>
+              <resolution>1</resolution>
+              <min_angle>-0.1</min_angle>
+              <max_angle>0.1</max_angle>
+            </horizontal>
+          </scan>
+          <range>
+            <min>0.04</min>
+            <max>0.30</max>
+            <resolution>0.001</resolution>
+          </range>
+        </lidar>
+        <always_on>1</always_on>
+        <visualize>true</visualize>
+        <topic>${topic}</topic>
+      </sensor>
+    </gazebo>
+  </xacro:macro>
+  <xacro:ir_gazebo name="ir_front_left"   topic="ir_front_left"/>
+  <xacro:ir_gazebo name="ir_front_center" topic="ir_front_center"/>
+  <xacro:ir_gazebo name="ir_front_right"  topic="ir_front_right"/>
   <gazebo>
     <plugin filename="gz-sim-diff-drive-system"
@@ -135,33 +158,4 @@
   <xacro:wheel_gazebo name="right_front_wheel"/>
   <xacro:wheel_gazebo name="right_rear_wheel"/>
-  <!-- IR Sensor Plugins -->
-  <xacro:macro name="ir_gazebo" params="name topic">
-    <gazebo reference="${name}">
-      <sensor name="${name}_sensor" type="gpu_lidar">
-        <update_rate>10</update_rate>
-        <lidar>
-          <scan>
-            <horizontal>
-              <samples>5</samples>
-              <resolution>1</resolution>
-              <min_angle>-0.1</min_angle>
-              <max_angle>0.1</max_angle>
-            </horizontal>
-          </scan>
-          <range>
-            <min>0.04</min>
-            <max>0.30</max>
-            <resolution>0.01</resolution>
-          </range>
-        </lidar>
-        <always_on>1</always_on>
-        <visualize>true</visualize>
-        <topic>${topic}</topic>
-      </sensor>
-    </gazebo>
-  </xacro:macro>
-  <xacro:ir_gazebo name="ir_front_left"   topic="ir_front_left"/>
-  <xacro:ir_gazebo name="ir_front_center" topic="ir_front_center"/>
-  <xacro:ir_gazebo name="ir_front_right"  topic="ir_front_right"/>
   <gazebo>
     <plugin filename="gz-sim-joint-state-publisher-system"

Commit message: fix: lower IR sensor height to 0.075m

File: slodda_description/urdf/slodda_real.urdf.xacro (robot description, xacro)
@@ -92,5 +92,5 @@
       <parent link="base_link"/>
       <child link="${name}"/>
-      <origin xyz="${x} ${y} 0.13" rpy="0 0 ${yaw}"/>
+      <origin xyz="${x} ${y} 0.075" rpy="0 0 ${yaw}"/>
     </joint>
   </xacro:macro>
