Commit message: feat: add Nav2 autonomous navigation with LD06 LiDAR
- Add LD06 LiDAR to URDF (lidar_link, fixed joint, gpu_lidar plugin)
- Fix DiffDrive child_frame_id: base_link -> base_footprint
- Add tf_topic to DiffDrive for correct odom->base_footprint TF
- Add /scan bridge to gazebo.launch.py
- Add arena_map.pgm + arena_map.yaml (78x53 @ 0.05m/px)
- Add nav2_params.yaml with RegulatedPurePursuit + /scan costmap
- Add nav2.launch.py with map_server, planner, controller, bt_navigator
- Fix enable_stamped_cmd_vel: false for Twist compatibility

File: slodda_description/urdf/slodda_real.urdf.xacro (robot description, xacro)
@@ -40,4 +40,56 @@
     </inertial>
   </link>
+<!-- LD06 LiDAR -->
+  <link name="lidar_link">
+    <visual>
+      <origin xyz="0 0 0" rpy="0 0 0"/>
+      <geometry>
+        <cylinder radius="0.019" length="0.033"/>
+      </geometry>
+      <material name="grey"/>
+    </visual>
+    <collision>
+      <origin xyz="0 0 0" rpy="0 0 0"/>
+      <geometry>
+        <cylinder radius="0.019" length="0.033"/>
+      </geometry>
+    </collision>
+    <inertial>
+      <mass value="0.180"/>
+      <origin xyz="0 0 0" rpy="0 0 0"/>
+      <inertia ixx="0.0001" ixy="0.0" ixz="0.0"
+               iyy="0.0001" iyz="0.0"
+               izz="0.0001"/>
+    </inertial>
+  </link>
+  <joint name="lidar_joint" type="fixed">
+    <parent link="base_link"/>
+    <child link="lidar_link"/>
+    <origin xyz="-0.05 0 0.122" rpy="0 0 0"/>
+  </joint>
+  <gazebo reference="lidar_link">
+    <sensor name="ld06_lidar" type="gpu_lidar">
+      <topic>scan</topic>
+      <gz_frame_id>lidar_link</gz_frame_id>
+      <update_rate>10</update_rate>
+      <lidar>
+        <scan>
+          <horizontal>
+            <samples>360</samples>
+            <resolution>1</resolution>
+            <min_angle>-3.14159</min_angle>
+            <max_angle>3.14159</max_angle>
+          </horizontal>
+        </scan>
+        <range>
+          <min>0.02</min>
+          <max>12.0</max>
+          <resolution>0.03</resolution>
+        </range>
+      </lidar>
+      <always_on>true</always_on>
+      <visualize>true</visualize>
+    </sensor>
+  </gazebo>
   <xacro:macro name="wheel" params="name x y">
     <link name="${name}">
@@ -144,5 +196,6 @@
       <odom_topic>odom</odom_topic>
       <frame_id>odom</frame_id>
-      <child_frame_id>base_link</child_frame_id>
+      <child_frame_id>base_footprint</child_frame_id>
+      <tf_topic>/tf</tf_topic>
     </plugin>
   </gazebo>

Commit message: fix: clock bridge, mesh orientation, TF direction, costmap sim_time, obstacle layer

File: slodda_description/urdf/slodda_real.urdf.xacro (robot description, xacro)
@@ -20,5 +20,5 @@
   <link name="base_link">
     <visual>
-      <origin xyz="0.1414 0.1000 0.0" rpy="${pi/2} 0 ${pi}"/>
+      <origin xyz="-0.1414 -0.1000 0.0" rpy="${pi/2} 0 0"/>
       <geometry>
         <mesh filename="package://slodda_description/meshes/chassis.stl" scale="0.001 0.001 0.001"/>
@@ -66,5 +66,5 @@
     <parent link="base_link"/>
     <child link="lidar_link"/>
-    <origin xyz="-0.05 0 0.122" rpy="0 0 0"/>
+    <origin xyz="0.05 0 0.122" rpy="0 0 0"/>
   </joint>
   <gazebo reference="lidar_link">
@@ -119,5 +119,5 @@
       <child link="${name}"/>
       <origin xyz="${x} ${y} 0" rpy="0 0 0"/>
-      <axis xyz="0 -1 0"/>
+      <axis xyz="0 1 0"/>
     </joint>
   </xacro:macro>
@@ -147,7 +147,7 @@
     </joint>
   </xacro:macro>
-  <xacro:ir_sensor name="ir_front_left"   x="-0.135" y=" 0.07" yaw="${pi - 0.3}"/>
-  <xacro:ir_sensor name="ir_front_center" x="-0.135" y=" 0.00" yaw="${pi}"/>
-  <xacro:ir_sensor name="ir_front_right"  x="-0.135" y="-0.07" yaw="${pi + 0.3}"/>
+  <xacro:ir_sensor name="ir_front_left"   x=" 0.135" y=" 0.07" yaw="0.3"/>
+  <xacro:ir_sensor name="ir_front_center" x=" 0.135" y=" 0.00" yaw="0"/>
+  <xacro:ir_sensor name="ir_front_right"  x=" 0.135" y="-0.07" yaw="-0.3"/>
   <!-- IR sensor plugins -->
   <xacro:macro name="ir_gazebo" params="name topic">

Commit message: Lagt til yolo_camera_test.py med 10-bit bayer unpacking

File: slodda_description/urdf/slodda_real.urdf.xacro (robot description, xacro)
@@ -18,8 +18,7 @@
     <origin xyz="0 0 ${wheel_radius}" rpy="0 0 0"/>
   </joint>
-  <!-- CHASSIS: enkel boks, ingen mesh -->
   <link name="base_link">
     <visual>
-      <origin xyz="0.1414 0.1000 0.0" rpy="${pi/2} 0 ${pi}"/>
+      <origin xyz="-0.1414 -0.1000 0.0" rpy="${pi/2} 0 0"/>
       <geometry>
         <mesh filename="package://slodda_description/meshes/chassis.stl" scale="0.001 0.001 0.001"/>
@@ -28,17 +27,69 @@
     </visual>
     <collision>
-      <origin xyz="0.1414 0.1000 0.0" rpy="${pi/2} 0 ${pi}"/>
-      <geometry>
-        <mesh filename="package://slodda_description/meshes/chassis.stl" scale="0.001 0.001 0.001"/>
+      <origin xyz="0 0 0.061" rpy="0 0 0"/>
+      <geometry>
+        <box size="${chassis_length} ${chassis_width} ${chassis_height}"/>
       </geometry>
     </collision>
     <inertial>
       <mass value="${chassis_mass}"/>
-      <origin xyz="0.1414 0.1000 0.0" rpy="${pi/2} 0 ${pi}"/>
-      <inertia ixx="0.052" ixy="0.0" ixz="0.0"
-               iyy="0.046" iyz="0.0"
-               izz="0.078"/>
+      <origin xyz="0 0 0.061" rpy="0 0 0"/>
+      <inertia ixx="0.0197" ixy="0.0" ixz="0.0"
+               iyy="0.0164" iyz="0.0"
+               izz="0.0309"/>
     </inertial>
   </link>
+<!-- LD06 LiDAR -->
+  <link name="lidar_link">
+    <visual>
+      <origin xyz="0 0 0" rpy="0 0 0"/>
+      <geometry>
+        <cylinder radius="0.019" length="0.033"/>
+      </geometry>
+      <material name="grey"/>
+    </visual>
+    <collision>
+      <origin xyz="0 0 0" rpy="0 0 0"/>
+      <geometry>
+        <cylinder radius="0.019" length="0.033"/>
+      </geometry>
+    </collision>
+    <inertial>
+      <mass value="0.180"/>
+      <origin xyz="0 0 0" rpy="0 0 0"/>
+      <inertia ixx="0.0001" ixy="0.0" ixz="0.0"
+               iyy="0.0001" iyz="0.0"
+               izz="0.0001"/>
+    </inertial>
+  </link>
+  <joint name="lidar_joint" type="fixed">
+    <parent link="base_link"/>
+    <child link="lidar_link"/>
+    <origin xyz="0.05 0 0.122" rpy="0 0 0"/>
+  </joint>
+  <gazebo reference="lidar_link">
+    <sensor name="ld06_lidar" type="gpu_lidar">
+      <topic>scan</topic>
+      <gz_frame_id>lidar_link</gz_frame_id>
+      <update_rate>10</update_rate>
+      <lidar>
+        <scan>
+          <horizontal>
+            <samples>360</samples>
+            <resolution>1</resolution>
+            <min_angle>-3.14159</min_angle>
+            <max_angle>3.14159</max_angle>
+          </horizontal>
+        </scan>
+        <range>
+          <min>0.02</min>
+          <max>12.0</max>
+          <resolution>0.03</resolution>
+        </range>
+      </lidar>
+      <always_on>true</always_on>
+      <visualize>true</visualize>
+    </sensor>
+  </gazebo>
   <xacro:macro name="wheel" params="name x y">
     <link name="${name}">
@@ -75,4 +126,5 @@
   <xacro:wheel name="right_front_wheel" x=" ${wheel_x_offset}" y="-${wheel_y_offset}"/>
   <xacro:wheel name="right_rear_wheel"  x="-${wheel_x_offset}" y="-${wheel_y_offset}"/>
+  <!-- IR sensor lenker - ingen preserveFixedJoint, slik at de lumpes inn i base_link -->
   <xacro:macro name="ir_sensor" params="name x y yaw">
     <link name="${name}">
@@ -81,13 +133,10 @@
         <material name="grey"/>
       </visual>
-      <collision>
-        <geometry><box size="0.02 0.01 0.01"/></geometry>
-      </collision>
       <inertial>
-        <mass value="0.01"/>
+        <mass value="0.001"/>
         <origin xyz="0 0 0"/>
-        <inertia ixx="0.00001" ixy="0.0" ixz="0.0"
-                 iyy="0.00001" iyz="0.0"
-                 izz="0.00001"/>
+        <inertia ixx="0.000001" ixy="0.0" ixz="0.0"
+                 iyy="0.000001" iyz="0.0"
+                 izz="0.000001"/>
       </inertial>
     </link>
@@ -95,14 +144,45 @@
       <parent link="base_link"/>
       <child link="${name}"/>
-      <origin xyz="${x} ${y} 0.04" rpy="0 0 ${yaw}"/>
+      <origin xyz="${x} ${y} 0.075" rpy="0 0 ${yaw}"/>
     </joint>
   </xacro:macro>
-  <xacro:ir_sensor name="ir_front_left"   x="-0.135" y=" 0.07" yaw=" 0.3"/>
-  <xacro:ir_sensor name="ir_front_center" x="-0.135" y=" 0.00" yaw=" 0.0"/>
-  <xacro:ir_sensor name="ir_front_right"  x="-0.135" y="-0.07" yaw="-0.3"/>
+  <xacro:ir_sensor name="ir_front_left"   x=" 0.135" y=" 0.07" yaw="0.3"/>
+  <xacro:ir_sensor name="ir_front_center" x=" 0.135" y=" 0.00" yaw="0"/>
+  <xacro:ir_sensor name="ir_front_right"  x=" 0.135" y="-0.07" yaw="-0.3"/>
+  <!-- IR sensor plugins -->
+  <xacro:macro name="ir_gazebo" params="name topic">
+    <gazebo reference="${name}">
+      <sensor name="${name}_sensor" type="gpu_lidar">
+        <update_rate>10</update_rate>
+        <lidar>
+          <scan>
+            <horizontal>
+              <samples>5</samples>
+              <resolution>1</resolution>
+              <min_angle>-0.1</min_angle>
+              <max_angle>0.1</max_angle>
+            </horizontal>
+          </scan>
+          <range>
+            <min>0.04</min>
+            <max>0.30</max>
+            <resolution>0.001</resolution>
+          </range>
+        </lidar>
+        <always_on>1</always_on>
+        <visualize>true</visualize>
+        <topic>${topic}</topic>
+      </sensor>
+    </gazebo>
+  </xacro:macro>
+  <xacro:ir_gazebo name="ir_front_left"   topic="ir_front_left"/>
+  <xacro:ir_gazebo name="ir_front_center" topic="ir_front_center"/>
+  <xacro:ir_gazebo name="ir_front_right"  topic="ir_front_right"/>
   <gazebo>
     <plugin filename="gz-sim-diff-drive-system"
             name="gz::sim::systems::DiffDrive">
+      <left_joint>left_front_wheel_joint</left_joint>
       <left_joint>left_rear_wheel_joint</left_joint>
+      <right_joint>right_front_wheel_joint</right_joint>
       <right_joint>right_rear_wheel_joint</right_joint>
       <wheel_separation>${wheel_y_offset * 2}</wheel_separation>
@@ -116,5 +196,6 @@
       <odom_topic>odom</odom_topic>
       <frame_id>odom</frame_id>
-      <child_frame_id>base_link</child_frame_id>
+      <child_frame_id>base_footprint</child_frame_id>
+      <tf_topic>/tf</tf_topic>
     </plugin>
   </gazebo>
@@ -130,3 +211,8 @@
   <xacro:wheel_gazebo name="right_front_wheel"/>
   <xacro:wheel_gazebo name="right_rear_wheel"/>
+  <gazebo>
+    <plugin filename="gz-sim-joint-state-publisher-system"
+            name="gz::sim::systems::JointStatePublisher">
+    </plugin>
+  </gazebo>
 </robot>
