Commit message: feat: YOLO teddy bear detection + Nav2 autonomous navigation
- Add yolo_detector node: YOLOv8n class-77 detection at 5 Hz, always
  streams /yolo/image so camera feed is live even between inference ticks
- Add bear_mission node: autonomous Nav2 goal to teddy bear position
- Add object_tracker node
- Add textured teddy bear Gazebo model with PNG albedo map
- Add nav2.rviz config: 3D orbit view, map/costmap/laserscan/YOLO camera
- Split Nav2 startup into two timer groups (localization 10 s, navigation
  15 s) to fix AMCL lifecycle timeout race condition
- Add bond_timeout=0.0 to both lifecycle managers
- Add LIBGL_ALWAYS_SOFTWARE=1 to RViz to fix NVIDIA GLSL segfault
- Add AMCL set_initial_pose at (0,0,0) in nav2_params.yaml
- Add *.pt to .gitignore

File: src/slodda_description/urdf/slodda_real.urdf.xacro (robot description, xacro)
@@ -216,3 +216,50 @@
     </plugin>
   </gazebo>
+  <!-- Camera (Raspberry Pi Camera v2 equivalent) -->
+  <link name="camera_link">
+    <visual>
+      <origin xyz="0 0 0" rpy="0 0 0"/>
+      <geometry>
+        <box size="0.03 0.03 0.03"/>
+      </geometry>
+      <material name="dark_grey"/>
+    </visual>
+    <collision>
+      <origin xyz="0 0 0" rpy="0 0 0"/>
+      <geometry>
+        <box size="0.03 0.03 0.03"/>
+      </geometry>
+    </collision>
+    <inertial>
+      <mass value="0.05"/>
+      <inertia ixx="1e-5" ixy="0" ixz="0" iyy="1e-5" iyz="0" izz="1e-5"/>
+    </inertial>
+  </link>
+  <joint name="camera_joint" type="fixed">
+    <parent link="base_link"/>
+    <child link="camera_link"/>
+    <origin xyz="0.1 0 0.15" rpy="0 0 0"/>
+  </joint>
+  <gazebo reference="camera_link">
+    <sensor name="camera" type="camera">
+      <pose>0 0 0 0 0 0</pose>
+      <topic>camera/image_raw</topic>
+      <gz_frame_id>camera_link</gz_frame_id>
+      <update_rate>30</update_rate>
+      <always_on>1</always_on>
+      <visualize>true</visualize>
+      <camera>
+        <horizontal_fov>1.085</horizontal_fov>
+        <image>
+          <width>640</width>
+          <height>480</height>
+          <format>R8G8B8</format>
+        </image>
+        <clip>
+          <near>0.05</near>
+          <far>20.0</far>
+        </clip>
+      </camera>
+    </sensor>
+  </gazebo>
 </robot>

Commit message: feat: autonomous bear mission with Nav2 override, tracking controller, and return-home
- mission_control: full state machine (IDLE → NAVIGATE → TRACK_BEAR → AT_BEAR → RETURN_HOME)
- Nav2 override: YOLO streak-gating (3 consecutive detections) cancels active Nav2 goal
  and transitions directly to TRACK_BEAR, preventing spurious triggers
- Tracking controller: two-phase approach (rotate-to-centre + LiDAR distance control)
  with drift correction, too-close detection, and LOST_TARGET recovery
- Return-home: odom waypoints recorded every 5 cm during navigation, replayed in reverse
  on APPROVE; robot drives back along its own path at 15 cm/s
- bear_mission: fix LiDAR fallback (distinguish too-close from out-of-range), fix
  overshoot deadlock (one-sided completion criterion), fix use_align_and_approach
  parameter ignored on CANCELING path, fix orphan Nav2 goal race condition, remove
  dead threading import and TASK_COMPLETE constant
- slodda_description: restore config/ install rule so view_real_robot.launch.py works
- slodda_rviz_panel: add custom RViz panel for mission control
- motor_driver_node + gpio_backend: hardware motor driver scaffold for real robot
- docs: full README rewrite with state machine diagram and topic table
- docs: CHEATSHEET.md with ROS2 / Git / Pi quick reference

File: src/slodda_description/urdf/slodda_real.urdf.xacro (robot description, xacro)
@@ -216,4 +216,37 @@
     </plugin>
   </gazebo>
+  <!-- IMU (BNO085 9-DOF equivalent) -->
+  <link name="imu_link">
+    <inertial>
+      <mass value="0.005"/>
+      <origin xyz="0 0 0"/>
+      <inertia ixx="1e-6" ixy="0" ixz="0" iyy="1e-6" iyz="0" izz="1e-6"/>
+    </inertial>
+  </link>
+  <joint name="imu_joint" type="fixed">
+    <parent link="base_link"/>
+    <child link="imu_link"/>
+    <origin xyz="0 0 0.061" rpy="0 0 0"/>
+  </joint>
+  <gazebo reference="imu_link">
+    <sensor name="imu_sensor" type="imu">
+      <topic>imu/data</topic>
+      <gz_frame_id>imu_link</gz_frame_id>
+      <update_rate>100</update_rate>
+      <always_on>true</always_on>
+      <imu>
+        <angular_velocity>
+          <x><noise type="gaussian"><mean>0</mean><stddev>0.009</stddev></noise></x>
+          <y><noise type="gaussian"><mean>0</mean><stddev>0.009</stddev></noise></y>
+          <z><noise type="gaussian"><mean>0</mean><stddev>0.009</stddev></noise></z>
+        </angular_velocity>
+        <linear_acceleration>
+          <x><noise type="gaussian"><mean>0</mean><stddev>0.021</stddev></noise></x>
+          <y><noise type="gaussian"><mean>0</mean><stddev>0.021</stddev></noise></y>
+          <z><noise type="gaussian"><mean>0</mean><stddev>0.021</stddev></noise></z>
+        </linear_acceleration>
+      </imu>
+    </sensor>
+  </gazebo>
   <!-- Camera (Raspberry Pi Camera v2 equivalent) -->
   <link name="camera_link">
